Commit message: Slam And Path Planning Bonus

File: luqman_bot/urdf/custom_bot.urdf (robot description, URDF)
Before this commit: robot luqman_bot, 6 links, 5 joints
Joints:
- joint left_wheel_joint: origin xyz=-0.2825 -0.125 -0.05 rpy=-1.5708 0.0 0.0 -> xyz=-0.2825 0.125 -0.05 rpy=-1.5708 0.0 0.0
- joint right_wheel_joint: origin xyz=-0.2825 0.125 -0.05 rpy=-1.5708 0.0 0.0 -> xyz=-0.2825 -0.125 -0.05 rpy=-1.5708 0.0 0.0
